File: rtc.brd (EAGLE design)
At the start: 27.9 x 29.2 mm, 19 parts, among them U1 MCP79412, U2 MCP980X, Y1 32.768 kHz

Commit message: v2.1
Parts:
- D1: device _jc:SOD-323F -> _jc:SOD-323F-A
- U1: value MCP79412 -> MCP7941x
Other:
- board text added: "jc 0414 v2.1"
- board text removed: "jc 0314 v2.0"
Changed lines of the file:
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@@
 <text x="19.05" y="7.62" size="1.4224" layer="22" ratio="16" rot="MR0">MCP7941x</text>
 <text x="22.86" y="5.715" size="1.4224" layer="22" ratio="16" rot="MR0">Real-Time Clock</text>
-<text x="21.59" y="3.81" size="1.4224" layer="22" ratio="16" rot="MR0">jc 0314 v2.0</text>
+<text x="21.59" y="3.81" size="1.4224" layer="22" ratio="16" rot="MR0">jc 0414 v2.1</text>
 <text x="19.05" y="1.905" size="1.4224" layer="22" ratio="16" rot="MR0">CC BY-SA</text>
 <text x="24.13" y="22.86" size="1.27" layer="21" ratio="16" rot="R90">79412</text>
@@
 </autorouter>
 <elements>
-<element name="U1" library="_jc" package="MSOP8" value="MCP79412" x="16.129" y="14.224" smashed="yes" rot="R180">
+<element name="U1" library="_jc" package="MSOP8" value="MCP7941x" x="16.129" y="14.224" smashed="yes" rot="R180">
 <attribute name="NAME" x="14.3256" y="13.6144" size="0.8128" layer="25" ratio="16" rot="R90"/>
 <attribute name="VALUE" x="13.589" y="16.129" size="0.8128" layer="27" ratio="16" rot="R270"/>
@@
 <attribute name="VALUE" x="5.715" y="2.54" size="1.27" layer="27" rot="R90"/>
 </element>
-<element name="D1" library="_jc" package="SOD-323F" value="PMEG6002EJ" x="2.5146" y="15.7734" smashed="yes" rot="R90">
-<attribute name="NAME" x="1.5638" y="15.1672" size="0.8128" layer="25" font="vector" ratio="16" rot="R90"/>
+<element name="D1" library="_jc" package="SOD-323F-A" value="PMEG6002EJ" x="2.5146" y="15.7734" smashed="yes" rot="R90">
+<attribute name="NAME" x="4.3578" y="15.1672" size="0.8128" layer="25" font="vector" ratio="16" rot="R90"/>
 <attribute name="VALUE" x="4.2146" y="13.6734" size="0.8128" layer="27" font="vector" ratio="16" rot="R90"/>
 </element>
@@
 </signal>
 </signals>
-<errors>
-</errors>
 </board>
 </drawing>
