File: rtc.sch (EAGLE design)
At the start: 19 parts, among them U1 MCP79412, U2 MCP980X, Y1 32.768 kHz

Commit message: v2.1
Parts:
- D1: device _jc:DIODESOD-323F -> _jc:DIODESOD-323F-A
- U1: value MCP79412 -> MCP7941x
Other:
- note added: "MCP7941x Breakout Board with Temperature Sensor by Jack Christensen"
- note added: "http://creativecommons.org/licenses/by-sa/4.0/"
- note added: "is licensed under CC BY-SA 4.0,"
- note added: "v2.1"
- note removed: "MCP79412 Breakout Board by Jack Christensen is licensed under"
- note removed: "a Creative Commons Attribution-ShareAlike 3.0 Unported License."
- note removed: "v1.2"
- moved on the sheet: JP1, JP2
